File: KiCad Files/Gremlin_v2.kicad_sch (KiCad schematic)
At the start: 57 parts, among them J1 JST_02, J2 JST_06, J3 JST_06, SW1 Switch, SW2 SW_SPST, U1 Nice_Nano_V2

Commit message: Added Scotto Libraries and created a new Gremlin v3 folder
Parts:
- removed D21, D22, D23, D24, D25: Diode, ScottoKeebs_Components:Diode_SOD-123, symbol Scotto:Placeholder_Diode
- removed J2, J3: JST_06, Connector_JST:JST_EH_B6B-EH-A_1x06_P2.50mm_Vertical, symbol PCM_SL_Connectors:JST_06
- removed S21: JS5208, ESwitch-JS5208:SW_JS5208, symbol E-Switch JS5208:JS5208
- removed SW3: ~, ProLib_pcs_2025-12-10:SW-TH_RKJXM1015001, symbol Gremlin:RKJXM1015001
- added J2: Conn_01x05, Connector_FFC-FPC:Molex_200528-0050_1x05-1MP_P1.00mm_Horizontal, symbol Connector_Generic:Conn_01x05
Connections:
- net NavSwitch is gone; now on net Row 0: U1.10 (D7)
- net Row 0: no longer U1.20 (D21)
- net Row 1: now also U1.11 (D8); no longer U1.19 (D20)
- net Row 2: now also U1.12 (D9); no longer U1.18 (D19)
- net Row 3: now also U1.14 (D16); no longer U1.17 (D18)
- net Row 4: now also U1.13 (D10); no longer U1.16 (D15)
- net at U1.21 (3.3v): now also J2.2 (Pin_2)
- net at SW1.1, U1.3 (GND): now also J2.5 (Pin_5)
- new net: J2.1 (Pin_1), U1.20 (D21)
- new net: J2.3 (Pin_3), U1.18 (D19)
- new net: J2.4 (Pin_4), U1.17 (D18)
